Commit message: Add files via upload

File: mani1_config/urdf/mani1_config.urdf (robot description, URDF)
Before this commit: robot mani1_config, 19 links, 18 joints
Joints:
- joint mani1_joint7: origin xyz=0 -0.3209 0 rpy=1.5708 2.6193E-32 0 -> xyz=0 -0.3209 0 rpy=1.5708 0 0
- joint mani2_joint7: origin xyz=0 -0.16398 0 rpy=1.5708 0 -1.2246E-16 -> xyz=0 -0.1745 0 rpy=1.5708 0 -1.2246E-16
